File: hw/NanoCurrentsSupply/NanoCurrentsSupply.kicad_sch (KiCad schematic)
At the start: 49 parts, among them J1 Conn_01x05_Pin, J2 Screw_Terminal_01x02, J3 Conn_02x03_Counter_Clockwise, J4 Conn_Coaxial, J5 Conn_Coaxial, U1 ADS1015IDGS, U2 INA240A1D, U3 LP2980-ADJ, U4 LP2980-ADJ, U5 LP2980-ADJ, U6 LP2980-ADJ, U7 LMV358

Commit message: Finished first PCB of NanoCurrentsSupply
Parts:
- Rs1: value R -> 1; footprint Resistor_SMD:R_4020_10251Metric_Pad1.65x5.30mm_HandSolder -> Resistor_SMD:R_1206_3216Metric_Pad1.30x1.75mm_HandSolder
Other:
- note added: "V_out = I * G * Rs I = 500mA max, 150 moy G = 20 (INA240A1) Rs = 1Ohms"
Changed lines of the file:
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@@
 		)
 	)
+	(text "V_out = I * G * Rs\nI = 500mA max, 150 moy\nG = 20 (INA240A1)\nRs = 1Ohms"
+		(exclude_from_sim no)
+		(at 121.666 94.488 0)
+		(effects
+			(font
+				(size 1.27 1.27)
+			)
+			(justify left)
+		)
+	)
 	(text "DUT out"
 		(exclude_from_sim no)
@@
 			)
 		)
-		(property "Value" "R"
+		(property "Value" "1"
 			(at 266.7 74.93 90)
 			(effects
@@
 			)
 		)
-		(property "Footprint" "Resistor_SMD:R_4020_10251Metric_Pad1.65x5.30mm_HandSolder"
+		(property "Footprint" "Resistor_SMD:R_1206_3216Metric_Pad1.30x1.75mm_HandSolder"
 			(at 266.7 72.898 90)
 			(effects

Commit message: Update HW before production
Parts:
- added D1: LED, LED_SMD:LED_0603_1608Metric, symbol Device:LED
- added R19: 200, Resistor_SMD:R_0603_1608Metric_Pad0.98x0.95mm_HandSolder, symbol Device:R
- C14, C16: now not fitted
- R15, R16: value ~ -> 0
Connections:
- net +5VP: now also R19.1
- net GND: now also D1.1 (K)
- new net: D1.2 (A), R19.2

Commit message: Rev B00 : only use one regulator
Parts:
- removed C10, C4, C7: 4.7uF, Capacitor_SMD:C_0603_1608Metric_Pad1.08x0.95mm_HandSolder, symbol Device:C
- removed C5, C8: 1uF, Capacitor_SMD:C_0603_1608Metric_Pad1.08x0.95mm_HandSolder, symbol Device:C
- removed C6, C9: 0.1uF, Capacitor_SMD:C_0603_1608Metric_Pad1.08x0.95mm_HandSolder, symbol Device:C
- removed J3: Conn_02x03_Counter_Clockwise, Connector_PinSocket_2.54mm:PinSocket_2x03_P2.54mm_Vertical, symbol Connector_Generic:Conn_02x03_Odd_Even
- removed R10, R7: 100k, Resistor_SMD:R_0603_1608Metric_Pad0.98x0.95mm_HandSolder, symbol Device:R
- removed U3, U4, U5: LP2980-ADJ, Package_TO_SOT_SMD:SOT-23-5, symbol Regulator_Linear:LP2980-ADJ
- added C1: 1uF, Capacitor_SMD:C_0603_1608Metric_Pad1.08x0.95mm_HandSolder, symbol Device:C
- added J2: Conn_02x03_Counter_Clockwise, Connector_PinSocket_2.54mm:PinSocket_2x03_P2.54mm_Vertical, symbol Connector_Generic:Conn_02x03_Odd_Even
- added U1: LP2980-ADJ, Package_TO_SOT_SMD:SOT-23-5, symbol Regulator_Linear:LP2980-ADJ
- C2: value 1uF -> 0.1uF
- C3: value 0.1uF -> 4.7uF
- renumbered C14 to C10, C16 to C11, C1 to C12, C11 to C4, C17 to C5, C18 to C6, C15 to C7, C12 to C8, C13 to C9, J2 to J1, J4 to J3, J5 to J4, J1 to J5, R3 to R1, R12 to R10, R13 to R11, R14 to R12, R15 to R13, R16 to R14, R19 to R15, R1 to R16, R2 to R17, R5 to R2, R6 to R3, R8 to R5, R9 to R6, R11 to R7, R17 to R8, R18 to R9, U6 to U2, U7 to U3, U2 to U4, U1 to U5
Connections:
- net +1V8 is gone; now on net RS_HIGH: R6.1, R7.1
- net +3.3V is gone; now on net RS_HIGH: R3.1, R5.1
- net +5V is gone; now on net RS_HIGH: C3.1, R1.1, R2.1
- net GND: now also C3.2, C1.2, U1.2 (GND); no longer C2.2
- net RS_HIGH: now also C2.1, U1.5 (VOUT)
- net VCC: now also C1.1, U1.1 (VIN), U1.3 (ON/~{OFF}); no longer C2.1
- net at R1.2, R2.2: now also J2.5 (Pin_5); no longer C3.2, R4.1
- net at R3.2, R5.2: now also J2.3 (Pin_3)
- net at R6.2, R7.2: now also J2.1 (Pin_1)
- new net FB_DIVIDER_OUT: C2.2, J2.2 (Pin_2), J2.4 (Pin_4), J2.6 (Pin_6), R4.1, U1.4 (ADJ)
Other:
- note added: "175k eq. for 3.3V"
- note added: "316k eq. for 5V"
- note added: "50k eq. for 1.8V"
- note removed: "175k eq."
- note removed: "50k eq."
- moved on the sheet: C10, C7, D1, J1, J3, J4, J5, R1, R13, R15, R2, R3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
